File: hardware/panasonic-p11-revH.kicad_pcb (KiCad board)
At the start: 2 copper layers, 50.5 x 18 mm, 10 parts, among them J1 1x4, J11 1.27_RA_8way, J2 1x4

Commit message: hardware: simplify back silk to 4 large legible lines
0.55-0.65mm text was too small to read on the delivered boards. Back now
carries only title/rev, the CNT 12V warning, and the repo URL (split over
two lines) at 1.0-1.1mm. Pinouts remain on the front silk and in the docs.

Co-Authored-By: Claude Opus 5 <noreply@anthropic.com>
Claude-Session: https://claude.ai/code/session_01BQkgfhAH12YMdeYMtUUmA3
Other:
- board text added: "CNT PIN4=12V NO CONNECT"
- board text added: "PANASONIC AC IF rev H"
- board text added: "esphome-panasonic-ac"
- board text added: "github.com/bl0ckstat/"
- board text removed: "CNT: CN-CNT 5p PIN4=12V NO CONN"
- board text removed: "D1: 1N5819 C1: 100uF/16V"
- board text removed: "J11: CN-WLAN (DNSK-P11) 1.27mm"
- board text removed: "J1: IO1 IO0 GND 3V3 (direct)"
- board text removed: "J2: IO10 IO7 GND 5V (in only)"
- board text removed: "LLC: BSS138 2-ch module 10.16mm"
- board text removed: "MCU: ESP32-C3 SuperMini"
- board text removed: "PANASONIC AC INTERFACE rev H"
- board text removed: "UART 9600 8E1 TX=IO3 RX=IO4"
- board text removed: "github.com/bl0ckstat/esphome-panasonic-ac"
Changed lines of the file:
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@@
 		)
 	)
-	(gr_text "github.com/bl0ckstat/esphome-panasonic-ac"
-		(at 31.2 38.15 0)
+	(gr_text "CNT PIN4=12V NO CONNECT"
+		(at 31.8 30.2 0)
 		(layer "B.SilkS")
 		(effects
 			(font
-				(size 0.55 0.55)
-				(thickness 0.11)
+				(size 1 1)
+				(thickness 0.18)
 			)
 			(justify mirror)
 		)
 	)
-	(gr_text "MCU: ESP32-C3 SuperMini"
-		(at 31.2 27.35 0)
+	(gr_text "github.com/bl0ckstat/"
+		(at 31.8 33.1 0)
 		(layer "B.SilkS")
 		(effects
 			(font
-				(size 0.6 0.6)
-				(thickness 0.11)
+				(size 1 1)
+				(thickness 0.18)
 			)
 			(justify mirror)
 		)
 	)
-	(gr_text "LLC: BSS138 2-ch module 10.16mm"
-		(at 31.2 28.7 0)
+	(gr_text "esphome-panasonic-ac"
+		(at 31.8 35.7 0)
 		(layer "B.SilkS")
 		(effects
 			(font
-				(size 0.6 0.6)
-				(thickness 0.11)
+				(size 1 1)
+				(thickness 0.18)
 			)
 			(justify mirror)
 		)
 	)
-	(gr_text "D1: 1N5819  C1: 100uF/16V"
-		(at 31.2 30.05 0)
+	(gr_text "PANASONIC AC IF  rev H"
+		(at 31.8 27.3 0)
 		(layer "B.SilkS")
 		(effects
 			(font
-				(size 0.6 0.6)
-				(thickness 0.11)
+				(size 1.1 1.1)
+				(thickness 0.18)
 			)
 			(justify mirror)
-		)
-	)
-	(gr_text "J11: CN-WLAN (DNSK-P11) 1.27mm"
-		(at 31.2 31.4 0)
-		(layer "B.SilkS")
-		(effects
-			(font
-				(size 0.6 0.6)
-				(thickness 0.11)
-			)
-			(justify mirror)
-		)
-	)
-	(gr_text "CNT: CN-CNT 5p PIN4=12V NO CONN"
-		(at 31.2 32.75 0)
-		(layer "B.SilkS")
-		(effects
-			(font
-				(size 0.6 0.6)
-				(thickness 0.11)
-			)
-			(justify mirror)
-		)
-	)
-	(gr_text "J1: IO1 IO0 GND 3V3 (direct)"
-		(at 31.2 34.1 0)
-		(layer "B.SilkS")
-		(effects
-			(font
-				(size 0.6 0.6)
-				(thickness 0.11)
-			)
-			(justify mirror)
-		)
-	)
-	(gr_text "J2: IO10 IO7 GND 5V (in only)"
-		(at 31.2 35.45 0)
-		(layer "B.SilkS")
-		(effects
-			(font
-				(size 0.6 0.6)
-				(thickness 0.11)
-			)
-			(justify mirror)
-		)
-	)
-	(gr_text "UART 9600 8E1 TX=IO3 RX=IO4"
-		(at 31.2 36.8 0)
-		(layer "B.SilkS")
-		(effects
-			(font
-				(size 0.6 0.6)
-				(thickness 0.11)
-			)
-			(justify mirror)
-		)
-	)
-	(gr_text "PANASONIC AC INTERFACE  rev H"
-		(at 31.2 26 0)
-		(layer "B.SilkS")
-		(effects
-			(font
-				(size 0.65 0.65)
-				(thickness 0.11)
-			)
-			(justify mirror)
